File: keyboard_keyboard.kicad_pcb (KiCad board)
At the start: 2 copper layers, 318 x 76.2 mm, 64 parts, among them K1 KEYSW, K10 KEYSW, K11 KEYSW, K12 KEYSW, K13 KEYSW, K14 KEYSW, K15 KEYSW, K16 KEYSW, K17 KEYSW, K18 KEYSW, K19 KEYSW, K2 KEYSW, K20 KEYSW, K21 KEYSW, K22 KEYSW, K23 KEYSW, K24 KEYSW, K25 KEYSW, K26 KEYSW, K27 KEYSW, K3 KEYSW, K4 KEYSW, K5 KEYSW, K6 KEYSW, K7 KEYSW, K8 KEYSW, K9 KEYSW, SW2 SW_PUSH, U1 ProMicro

Commit message: Second iteration of design
Still based on the pro micro, but smaller PCB with more knobs and mod keys!
Parts:
- removed R1: 10k, Resistor_THT:R_Axial_DIN0204_L3.6mm_D1.6mm_P5.08mm_Horizontal
- added D28: D, keyboard_parts:D_SOD123_axial, F.Cu at (109.5, 90.7)
- added D29: D, keyboard_parts:D_SOD123_axial, F.Cu at (128.5, 90.7)
- added K28: KEYSW, Button_Switch_Keyboard:SW_Cherry_MX_1.00u_PCB, F.Cu at (102.4, 84.3)
- added K29: KEYSW, Button_Switch_Keyboard:SW_Cherry_MX_1.00u_PCB, F.Cu at (121.4, 84.3)
- added RV3: R_POT, Potentiometer_THT:Potentiometer_Omeg_PC16BU_Vertical, F.Cu at (238.3, 98.3)
- moved D27 76.4 mm to (80.8, 90.7), turned to 90 degrees
- moved D26 74.1 mm to (61.7, 90.7), turned to 90 degrees
- moved K27 69.0 mm to (73.7, 84.3)
- moved K26 60.4 mm to (54.6, 84.3)
- moved H1 30.0 mm to (28.2, 77.5)
- moved H3 30.0 mm to (28.2, 143.5)
- moved D11 21.1 mm to (147.6, 115.3), turned to 90 degrees
- moved D14 21.1 mm to (185.7, 115.3), turned to 90 degrees
- moved D19 21.1 mm to (242.8, 115.3), turned to 90 degrees
- moved D21 21.1 mm to (261.9, 115.3), turned to 90 degrees
- moved D2 21.1 mm to (52.3, 115.3), turned to 90 degrees
- moved D7 21.1 mm to (109.5, 115.3), turned to 90 degrees
- moved D9 21.1 mm to (128.5, 115.3), turned to 90 degrees
- moved D4 21.1 mm to (71.4, 115.3), turned to 90 degrees
- moved D16 21.1 mm to (204.7, 115.3), turned to 90 degrees
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- renumbered SW2 to SW1
Connections:
- D26 pad 1: Row3 -> ModRow
- D27 pad 1: Row3 -> ModRow
- K26 pad 1: Col7 -> Col1
- K27 pad 1: Col8 -> Col2
- U1 pad 5: (no net) -> ModRow
- U1 pad 6: (no net) -> Row1
- U1 pad 7: Row1 -> Row2
- U1 pad 8: Row2 -> Row3
- U1 pad 9: Row3 -> Pot3
Routing:
- net Col8: track 358.6 -> 24.6 mm
- net ModRow: track 0.00 -> 226.9 mm
- net Row3: track 327.7 -> 123.2 mm, vias 0 -> 1
- net Col7: track 334.7 -> 176.3 mm, vias 1 -> 0
- net Col3: track 254.0 -> 315.2 mm, vias 3 -> 1
- net Pot3: track 0.00 -> 54.0 mm
- net VCC: track 0.00 -> 29.4 mm
- net Col4: track 279.6 -> 298.5 mm, vias 0 -> 1
- net Pot2: track 73.1 -> 91.6 mm
- net Row4: track 180.8 -> 162.8 mm, vias 1 -> 0
- net Col1: track 344.3 -> 362.1 mm, vias 0 -> 1
- net Col6: track 236.1 -> 218.7 mm, vias 0 -> 1
- net Col5: track 258.3 -> 242.1 mm, vias 0 -> 1
- net Col2: track 323.1 -> 339.0 mm, vias 0 -> 1
- net Row1: track 244.8 -> 260.1 mm, vias 1 -> 0
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- added copper zone on B.Cu, net GND
- added copper zone on F.Cu, net VCC
- removed copper zone on F.Cu, net GND
- removed copper zone on B.Cu, net VCC
Other:
- board size 318 x 76.2 mm -> 286 x 76.2 mm
